File: shield-attiny/shield-attiny.sch (KiCad schematic (older format))
At the start: 9 parts, among them SW1 SW_Push, U1 ATtiny85-20PU

Commit message: Adiconando Layout
Parts:
- removed D1: LED_RGBC, LED_THT:LED_D5.0mm-4_RGB, symbol Device:LED_RGBC
- added D1: LED_RCBG, LED_THT:LED_D5.0mm-4_RGB, symbol Device:LED_RCBG
- A1: footprint Module:Arduino_UNO_R3 -> shield-attiny:Arduino_UNO_R3
Connections:
- net GND: now also D1.2 (K)
- net at R2.2: now also D1.1 (RA)
- net at R3.2: now also D1.4 (GA)
- net at R4.2: now also D1.3 (BA)
- no-connect marks 2 -> 21
Changed lines of the file:
@@
 Rev "1.0"
 Comp "Franzininho"
-Comment1 ""
+Comment1 "Fábio"
 Comment2 ""
 Comment3 ""
@@
 F 0 "A1" H 8350 4131 50  0000 C CNN
 F 1 "Arduino_UNO_R3" H 8350 4040 50  0000 C CNN
-F 2 "Module:Arduino_UNO_R3" H 8350 2950 50  0001 C CIN
+F 2 "shield-attiny:Arduino_UNO_R3" H 8350 2950 50  0001 C CIN
 F 3 "https://www.arduino.cc/en/Main/arduinoBoardUno" H 8350 2950 50  0001 C CNN
 	1    8350 2950
@@
 	4050 3600 4050 3750
 $Comp
-L Device:LED_RGBC D1
-U 1 1 603047DD
-P 5850 2900
-F 0 "D1" H 5850 3397 50  0000 C CNN
-F 1 "LED_RGBC" H 5850 3306 50  0000 C CNN
-F 2 "LED_THT:LED_D5.0mm-4_RGB" H 5850 2850 50  0001 C CNN
-F 3 "~" H 5850 2850 50  0001 C CNN
-	1    5850 2900
-	1    0    0    -1
-$EndComp
-$Comp
 L Device:R_US R4
 U 1 1 60308CC4
@@
 	6050 3100 6350 3100
 Wire Wire Line
-	9100 3750 8850 3750
-Wire Wire Line
 	9500 3750 9600 3750
 Wire Wire Line
 	9600 3750 9600 3950
+NoConn ~ 7850 2850
+NoConn ~ 7850 2750
+NoConn ~ 7850 2650
+NoConn ~ 7850 2550
+NoConn ~ 7850 2450
+NoConn ~ 7850 2350
+NoConn ~ 8850 3650
+NoConn ~ 8850 3450
+NoConn ~ 8850 3350
+NoConn ~ 8850 3250
+NoConn ~ 8850 3150
+NoConn ~ 8850 3050
+NoConn ~ 8850 2950
+NoConn ~ 8850 2750
+NoConn ~ 8850 2550
+NoConn ~ 8850 2350
+NoConn ~ 8550 1950
+NoConn ~ 8450 1950
+NoConn ~ 8250 1950
+Wire Wire Line
+	8850 3750 9100 3750
+$Comp
+L Device:LED_RCBG D1
+U 1 1 60414663
+P 5850 2900
+F 0 "D1" H 5850 3397 50  0000 C CNN
+F 1 "LED_RCBG" H 5850 3306 50  0000 C CNN
+F 2 "LED_THT:LED_D5.0mm-4_RGB" H 5850 2850 50  0001 C CNN
+F 3 "~" H 5850 2850 50  0001 C CNN
+	1    5850 2900
+	1    0    0    -1
+$EndComp
 $EndSCHEMATC
